File: Minisumo_EDU_1/Hardware/main.brd (EAGLE design)
At the start: 94 x 65 mm, 51 parts, among them Q1 IRFR5305

Commit message: V1.0 No software
Parts:
- C1, C10, C13, C14, C15, C16, C17, C18, C2, C3, C4, C5, C6, C7, C8, C9: value (none) -> 100nF
- C11, C12: value (none) -> 47uF
- R1, R15, R2, R5: value (none) -> 10K
- R16: value (none) -> 1K
- R3, R4: value (none) -> 4K7
- R6: value (none) -> 100R
- renumbered R7 to R15, R8 to R16
Routing:
- net BATT_LVL: track 36.8 -> 35.3 mm
Other:
- board text added: "MINISUMO_EDU_1"
- board text added: "MINISUMO_EDU_1_V1.00"
- board text added: "V1.00 1.03.2020 By zuba1"
- board text added: "ZUBA-projects"
- board text added: "github.com/ZUBA-projects/MINISUMO_ROBOT"
