File: Minisumo_EDU_1/Hardware/main.sch (EAGLE design)
At the start: 49 parts, among them Q1 IRFR5305

Commit message: V1.0 No software
Parts:
- removed R7, R8: (no value), rcl:R-EU_M0805
- added R15: 10K, rcl:R-EU_M0805
- added R16: 1K, rcl:R-EU_M0805
- C1, C10, C13, C14, C15, C16, C17, C18, C2, C3, C4, C5, C6, C7, C8, C9: value (none) -> 100nF
- C11, C12: value (none) -> 47uF
- R1, R2, R5: value (none) -> 10K
- R3, R4: value (none) -> 4K7
- R6: value (none) -> 100R
Connections:
- net BATT_LVL: now also R15.1, R16.2; no longer R7.1, R8.2
- net GND: now also R16.1; no longer R8.1
- net V+: now also R15.2; no longer R7.2
Other:
- moved on the sheet: AKU, B+, B-, BALANCER, C1, C10, C11, C13, C14, C15, C16, C18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
